File: Vehicle_car.kicad_pcb (KiCad board)
At the start: 2 copper layers, 35 parts, among them P1 SWD, P2 GPS, P3 SUPPLY, P4 COLOR_1, P5 COLOR_2, P6 MOTOR 1, P7 MOTOR 2, P8 BLUETOOTH, P9 GND, SW1 SW_PUSH_4PIN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

Commit message: Finished schematic. Not checked yet
Parts:
- added P10: Length_sen, PIN_ARRAY_4x1, F.Cu at (38.1, 44.5)
- moved U3 62.5 mm to (57.1, 67.3)
Connections:
- U3 pad 57: (no net) -> SEN_OUT
- U3 pad 58: (no net) -> SEN_EN
Changed lines of the file:
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@@
 (kicad_pcb (version 3) (host pcbnew "(2013-07-07 BZR 4022)-stable")
   (general
-    (links 110)
-    (no_connects 110)
-    (area 15.874999 11.3538 105.730674 68.852466)
+    (links 114)
+    (no_connects 114)
+    (area 0 0 0 0)
     (thickness 1.6)
     (drawings 0)
     (tracks 0)
     (zones 0)
-    (modules 35)
-    (nets 42)
+    (modules 36)
+    (nets 44)
   )
   (page A3)
@@
   (net 20 LED3)
   (net 21 LED4)
-  (net 22 N-0000015)
-  (net 23 N-0000016)
-  (net 24 N-0000017)
-  (net 25 N-0000023)
-  (net 26 N-0000070)
-  (net 27 N-0000073)
+  (net 22 N-0000018)
+  (net 23 N-0000023)
+  (net 24 N-0000024)
+  (net 25 N-0000025)
+  (net 26 N-0000052)
+  (net 27 N-0000066)
   (net 28 NRST)
   (net 29 OSC_IN)
@@
   (net 37 S1a)
   (net 38 S1b)
-  (net 39 SWDCLK)
-  (net 40 SWDIO)
-  (net 41 SWDO)
+  (net 39 SEN_EN)
+  (net 40 SEN_OUT)
+  (net 41 SWDCLK)
+  (net 42 SWDIO)
+  (net 43 SWDO)
   (net_class Default "To jest domyślna klasa połączeń."
     (clearance 0.254)
@@
     (add_net LED3)
     (add_net LED4)
-    (add_net N-0000015)
-    (add_net N-0000016)
-    (add_net N-0000017)
+    (add_net N-0000018)
     (add_net N-0000023)
-    (add_net N-0000070)
-    (add_net N-0000073)
+    (add_net N-0000024)
+    (add_net N-0000025)
+    (add_net N-0000052)
+    (add_net N-0000066)
     (add_net NRST)
     (add_net OSC_IN)
@@
     (add_net S1a)
     (add_net S1b)
+    (add_net SEN_EN)
+    (add_net SEN_OUT)
     (add_net SWDCLK)
     (add_net SWDIO)
@@
     (pad 2 smd rect (at 1.651 0) (size 1.524 2.032)
       (layers Gorna Pasty_Gorna Maski_Gorna)
-      (net 24 N-0000017)
+      (net 22 N-0000018)
     )
     (model smd/chip_cms.wrl
@@
     (pad 1 smd rect (at -1.651 0) (size 1.524 2.032)
       (layers Gorna Pasty_Gorna Maski_Gorna)
-      (net 24 N-0000017)
+      (net 22 N-0000018)
     )
     (pad 2 smd rect (at 1.651 0) (size 1.524 2.032)
@@
     (pad 2 smd rect (at 1.651 0) (size 1.524 2.032)
       (layers Gorna Pasty_Gorna Maski_Gorna)
-      (net 22 N-0000015)
+      (net 25 N-0000025)
     )
     (model smd/chip_cms.wrl
@@
     (pad 1 smd rect (at -1.651 0) (size 1.524 2.032)
       (layers Gorna Pasty_Gorna Maski_Gorna)
-      (net 22 N-0000015)
+      (net 25 N-0000025)
     )
     (pad 2 smd rect (at 1.651 0) (size 1.524 2.032)
@@
     (pad 2 smd rect (at 1.651 0) (size 1.524 2.032)
       (layers Gorna Pasty_Gorna Maski_Gorna)
-      (net 23 N-0000016)
+      (net 24 N-0000024)
     )
     (model smd/chip_cms.wrl
@@
     (pad 1 smd rect (at -1.651 0) (size 1.524 2.032)
       (layers Gorna Pasty_Gorna Maski_Gorna)
-      (net 23 N-0000016)
+      (net 24 N-0000024)
     )
     (pad 2 smd rect (at 1.651 0) (size 1.524 2.032)
@@
     (pad 2 smd rect (at 1.651 0) (size 1.524 2.032)
       (layers Gorna Pasty_Gorna Maski_Gorna)
-      (net 25 N-0000023)
+      (net 23 N-0000023)
     )
     (model smd/chip_cms.wrl
@@
     (pad 1 smd rect (at -1.651 0) (size 1.524 2.032)
       (layers Gorna Pasty_Gorna Maski_Gorna)
-      (net 25 N-0000023)
+      (net 23 N-0000023)
     )
     (pad 2 smd rect (at 1.651 0) (size 1.524 2.032)
@@
     (pad 2 smd rect (at 1.651 0) (size 1.524 2.032)
       (layers Gorna Pasty_Gorna Maski_Gorna)
-      (net 27 N-0000073)
+      (net 26 N-0000052)
     )
     (model smd/chip_cms.wrl
@@
     (pad 1 smd rect (at -1.651 0) (size 1.524 2.032)
       (layers Gorna Pasty_Gorna Maski_Gorna)
-      (net 26 N-0000070)
+      (net 27 N-0000066)
     )
     (pad 2 smd rect (at 1.651 0) (size 1.524 2.032)
@@
     (pad 2 smd rect (at 1.651 0) (size 1.524 2.032)
       (layers Gorna Pasty_Gorna Maski_Gorna)
-      (net 26 N-0000070)
+      (net 27 N-0000066)
     )
     (model smd/chip_cms.wrl
@@
     (pad 2 thru_hole circle (at -3.81 0) (size 1.524 1.524) (drill 1.016)
       (layers *.Cu *.Mask Opisowa_Gorna)
-      (net 39 SWDCLK)
+      (net 41 SWDCLK)
     )
     (pad 3 thru_hole circle (at -1.27 0) (size 1.524 1.524) (drill 1.016)
@@
     (pad 4 thru_hole circle (at 1.27 0) (size 1.524 1.524) (drill 1.016)
       (layers *.Cu *.Mask Opisowa_Gorna)
-      (net 40 SWDIO)
+      (net 42 SWDIO)
     )
     (pad 5 thru_hole circle (at 3.81 0) (size 1.524 1.524) (drill 1.016)
@@
     (pad 6 thru_hole circle (at 6.35 0) (size 1.524 1.524) (drill 1.016)
       (layers *.Cu *.Mask Opisowa_Gorna)
-      (net 41 SWDO)
+      (net 43 SWDO)
     )
     (model pin_array/pins_array_6x1.wrl
@@
   )
   (module LQFP64 (layer Gorna)
-    (at 111.76 36.83)
+    (at 57.15 67.31)
     (fp_text reference U3 (at 0 1.27) (layer Opisowa_Gorna)
       (effects (font (size 1.27 1.27) (thickness 0.2)))
@@
     (pad 46 smd rect (at 5.75 -2.75) (size 1.2 0.3)
       (layers Gorna Pasty_Gorna Maski_Gorna)
-      (net 40 SWDIO)
+      (net 42 SWDIO)
     )
     (pad 56 smd rect (at 0.25 -5.75 90) (size 1.2 0.3)
@@
     (pad 55 smd rect (at 0.75 -5.75 90) (size 1.2 0.3)
       (layers Gorna Pasty_Gorna Maski_Gorna)
-      (net 41 SWDO)
+      (net 43 SWDO)
     )
     (pad 54 smd rect (at 1.25 -5.75 90) (size 1.2 0.3)
@@
     (pad 57 smd rect (at -0.25 -5.75 90) (size 1.2 0.3)
       (layers Gorna Pasty_Gorna Maski_Gorna)
+      (net 40 SEN_OUT)
     )
     (pad 58 smd rect (at -0.75 -5.75 90) (size 1.2 0.3)
       (layers Gorna Pasty_Gorna Maski_Gorna)
+      (net 39 SEN_EN)
     )
     (pad 59 smd rect (at -1.25 -5.75 90) (size 1.2 0.3)
@@
     (pad 60 smd rect (at -1.75 -5.75 90) (size 1.2 0.3)
       (layers Gorna Pasty_Gorna Maski_Gorna)
-      (net 27 N-0000073)
+      (net 26 N-0000052)
     )
     (pad 61 smd rect (at -2.25 -5.75 90) (size 1.2 0.3)
@@
     (pad 49 smd rect (at 3.75 -5.75 90) (size 1.2 0.3)
       (layers Gorna Pasty_Gorna Maski_Gorna)
-      (net 39 SWDCLK)
+      (net 41 SWDCLK)
     )
     (pad 63 smd rect (at -3.25 -5.75 90) (size 1.2 0.3)
@@
       (at (xyz 0 0 0))
       (scale (xyz 1 1 1))
+      (rotate (xyz 0 0 0))
+    )
+  )
+  (module PIN_ARRAY_4x1 (layer Gorna)
+    (at 38.1 44.45 270)
+    (descr "Double rangee de contacts 2 x 5 pins")
+    (tags CONN)
+    (fp_text reference P10 (at 0 -2.54 270) (layer Opisowa_Gorna)
+      (effects (font (size 1.016 1.016) (thickness 0.2032)))
+    )
+    (fp_text value Length_sen (at 0 2.54 270) (layer Opisowa_Gorna) hide
+      (effects (font (size 1.016 1.016) (thickness 0.2032)))
+    )
+    (fp_line (start 5.08 1.27) (end -5.08 1.27) (layer Opisowa_Gorna) (width 0.254))
+    (fp_line (start 5.08 -1.27) (end -5.08 -1.27) (layer Opisowa_Gorna) (width 0.254))
+    (fp_line (start -5.08 -1.27) (end -5.08 1.27) (layer Opisowa_Gorna) (width 0.254))
+    (fp_line (start 5.08 1.27) (end 5.08 -1.27) (layer Opisowa_Gorna) (width 0.254))
+    (pad 1 thru_hole rect (at -3.81 0 270) (size 1.524 1.524) (drill 1.016)
+      (layers *.Cu *.Mask Opisowa_Gorna)
+      (net 39 SEN_EN)
+    )
+    (pad 2 thru_hole circle (at -1.27 0 270) (size 1.524 1.524) (drill 1.016)
+      (layers *.Cu *.Mask Opisowa_Gorna)
+      (net 40 SEN_OUT)
+    )
+    (pad 3 thru_hole circle (at 1.27 0 270) (size 1.524 1.524) (drill 1.016)
+      (layers *.Cu *.Mask Opisowa_Gorna)
+      (net 1 +3.3V)
+    )
+    (pad 4 thru_hole circle (at 3.81 0 270) (size 1.524 1.524) (drill 1.016)
+      (layers *.Cu *.Mask Opisowa_Gorna)
+      (net 15 GND)
+    )
+    (model pin_array\pins_array_4x1.wrl
+      (at (xyz 0 0 0))
+      (scale (xyz 1 1 1))

Commit message: PCB dimension
Parts:
- added DR1: DRILL_6MM_3MM, DRILL_6mm_3mm, F.Cu at (212.2, 124.8)
- added P11: GND, PIN_ARRAY_1, F.Cu at (259.0, 108.5)
- moved SW1 264.3 mm to (268.0, 145.0), turned to 90 degrees
- moved C7 248.6 mm to (268.0, 138.5)
- moved P10 242.1 mm to (270.0, 114.0)
- moved R7 235.7 mm to (268.0, 151.5)
- moved C6 233.8 mm to (239.0, 138.0), turned to 135 degrees
- moved R8 233.6 mm to (246.5, 122.0), turned to 225 degrees
- moved R3 230.0 mm to (215.5, 142.5), turned to 90 degrees
- moved C5 226.9 mm to (235.0, 142.0), turned to 135 degrees
- moved D4 226.2 mm to (213.0, 135.5), turned to 90 degrees
- moved R2 225.5 mm to (218.0, 142.5), turned to 90 degrees
- moved R4 225.3 mm to (213.5, 142.5), turned to 90 degrees
- moved D3 223.5 mm to (215.5, 135.5), turned to 90 degrees
- moved D2 218.7 mm to (218.0, 135.5), turned to 90 degrees
- moved U2 218.2 mm to (245.0, 145.0), turned to 45 degrees
- moved C8 216.2 mm to (245.5, 111.5), turned to 315 degrees
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Other:
- board text added: "NAPED"
- board text added: "SKRET"
