File: Vehicle_car.kicad_pcb (KiCad board)
At the start: 2 copper layers, 43 parts, among them P1 SWD, P10 Length_sen, P11 GND, P2 GPS, P3 SUPPLY, P4 COLOR_1, P5 COLOR_2, P6 MOTOR 1, P7 MOTOR 2, P8 BLUETOOTH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

Commit message: Started connect pads
Parts:
- removed D2, D3: GREEN, SM1206
- removed D4, D5: BLUE, SM1206
- removed R2, R3: 330R, SM1206
- removed R4, R5: 660R, SM1206
- C10, C11, C12, C13, C14, C3, C5, C6, C8, C9: moved to B.Cu
- SW1: value SW_PUSH_4PIN -> RESET
- moved P9 72.3 mm to (270.0, 114.5)
- moved P11 64.9 mm to (199.9, 140.3)
- moved P8 45.1 mm to (259.6, 126.0), turned to 270 degrees
- moved X1 42.1 mm to (237.3, 144.7), turned to 0 degrees
- moved U2 38.2 mm to (229.4, 110.1), turned to 180 degrees
- moved C9 30.4 mm to (234.2, 138.5), turned to 270 degrees
- moved P4 29.4 mm to (215.0, 100.0)
- moved C5 28.7 mm to (226.8, 113.5), turned to 270 degrees
- moved C8 26.5 mm to (237.2, 138.5), turned to 270 degrees
- moved C6 25.9 mm to (229.5, 113.5), turned to 270 degrees
- moved C12 24.6 mm to (240.2, 138.5), turned to 90 degrees
- moved C14 23.1 mm to (232.5, 113.5), turned to 270 degrees
- moved R8 21.7 mm to (226.2, 134.0), turned to 0 degrees
- moved C10 21.7 mm to (243.2, 130.2), turned to 180 degrees
- moved P5 19.8 mm to (215.0, 145.0), turned to 180 degrees
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Connections:
- C8 pad 2: OSC_IN -> OSC_OUT
- C9 pad 2: OSC_OUT -> OSC_IN
- P2 pad 3: (no net) -> +3.3V
- P8 pad 4: BLUETOOTH_RX -> BLUETOOTH_TX
- P8 pad 5: BLUETOOTH_TX -> BLUETOOTH_RX
- U3 pad 33: LED1 -> (no net)
- U3 pad 34: LED2 -> (no net)
- U3 pad 35: LED3 -> (no net)
- U3 pad 36: LED4 -> (no net)
- U3 pad 42: BLUETOOTH_TX -> BLUETOOTH_RX
- U3 pad 43: BLUETOOTH_RX -> BLUETOOTH_TX
- X1 pad 1: OSC_OUT -> OSC_IN
- X1 pad 2: OSC_IN -> OSC_OUT
Routing:
- net AO2: track 0.00 -> 50.9 mm
- net AO1: track 0.00 -> 50.1 mm
- net BO2: track 0.00 -> 40.3 mm
- net BO1: track 0.00 -> 38.9 mm
- net +9V: track 0.00 -> 28.3 mm, vias 0 -> 2
- net +3.3V: track 0.00 -> 26.7 mm, vias 0 -> 1
- net GND: track 0.00 -> 25.4 mm
- net N-0000063: track 0.00 -> 4.16 mm
Other:
- board outline added: 75 x 51 mm

Commit message: Finish PCB
Parts:
- C10, C11, C13, C3: moved to F.Cu
- SW1: value RESET -> SW_PUSH_4PIN
- moved C12 13.0 mm to (241.0, 125.6)
- moved C3 12.3 mm to (235.7, 114.8), turned to 90 degrees
- moved C10 11.5 mm to (250.6, 121.3), turned to 0 degrees
- moved C13 9.71 mm to (250.6, 127.6), turned to 0 degrees
- moved C8 9.25 mm to (246.2, 136.3)
- moved X1 8.30 mm to (237.4, 136.4)
- moved U3 7.73 mm to (239.1, 125.1)
- moved R8 7.30 mm to (227.7, 126.8)
- moved C11 6.23 mm to (227.7, 129.8), turned to 180 degrees
- moved C9 6.05 mm to (228.6, 136.3)
- moved C14 4.81 mm to (233.2, 108.8), turned to 90 degrees
- moved C5 4.78 mm to (226.2, 108.8), turned to 90 degrees
- moved C6 4.76 mm to (229.8, 108.8), turned to 90 degrees
Connections:
- U3 pad 1: (no net) -> +3.3V
Routing:
- net GND: track 25.4 -> 374.6 mm, vias 0 -> 24
- net +3.3V: track 26.7 -> 319.4 mm, vias 1 -> 16
- net OUTa: track 0.00 -> 102.8 mm, vias 0 -> 5
- net S0a: track 0.00 -> 88.9 mm, vias 0 -> 5
- net S1a: track 0.00 -> 72.0 mm, vias 0 -> 1
- net LEDa: track 0.00 -> 68.0 mm, vias 0 -> 5
- net OUTb: track 0.00 -> 63.0 mm, vias 0 -> 2
- net S0b: track 0.00 -> 61.9 mm, vias 0 -> 3
- net LEDb: track 0.00 -> 60.2 mm, vias 0 -> 1
- net NRST: track 0.00 -> 56.2 mm
- net S1b: track 0.00 -> 52.2 mm, vias 0 -> 1
- net SWDO: track 0.00 -> 52.0 mm, vias 0 -> 2
- net SWDIO: track 0.00 -> 51.9 mm, vias 0 -> 4
- net SWDCLK: track 0.00 -> 49.6 mm, vias 0 -> 4
- net PWMA: track 0.00 -> 41.3 mm, vias 0 -> 2
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Other:
- rule trace_min: 0.254 -> 0.1778

Commit message: ...
Parts:
- SW1: value SW_PUSH_4PIN -> RESET
- U3: value STM32F100RB -> STM32F100
Routing:
- net S0a: track 88.9 -> 90.2 mm
- added copper zone on B.Cu, net GND
- added copper zone on F.Cu, net GND
Other:
- rule trace_min: 0.1778 -> 0.254
- board text removed: "NAPED"
- board text removed: "SKRET"
- board text removed: "not fitted"
