File: Vehicle_car.kicad_pcb (KiCad board)
At the start: 2 copper layers, 75 x 51 mm, 35 parts, among them P1 SWD, P10 Length_sen, P11 GND, P2 GPS, P3 SUPPLY, P4 COLOR_1, P5 COLOR_2, P6 MOTOR 1, P7 MOTOR 2, P8 BLUETOOTH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

Commit message: generate gerber
Routing:
- net LEDb: track 60.2 -> 56.3 mm
- net OUTa: track 102.8 -> 103.6 mm
Changed lines of the file:
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@@
     (thickness 1.6)
     (drawings 8)
-    (tracks 1017)
+    (tracks 1023)
     (zones 0)
     (modules 35)
@@
   (layers
     (15 Gorna signal)
-    (0 Dolna signal hide)
+    (0 Dolna signal)
     (16 B.Adhes user)
     (17 F.Adhes user)
@@
   )
   (setup
-    (last_trace_width 0.508)
+    (last_trace_width 0.254)
     (user_trace_width 0.254)
     (user_trace_width 0.508)
@@
     (visible_elements 7FFFFFFF)
     (pcbplotparams
-      (layerselection 3178497)
+      (layerselection 284196865)
       (usegerberextensions true)
       (excludeedgelayer true)
@@
       (drillshape 0)
       (scaleselection 1)
-      (outputdirectory ""))
+      (outputdirectory gerbers/))
   )
   (net 0 "")
@@
   (segment (start 246.125 125.35) (end 246.65 125.875) (width 0.254) (layer Gorna) (net 16))
   (segment (start 246.65 125.875) (end 246.65 125.85) (width 0.254) (layer Dolna) (net 16))
+  (segment (start 207.38 145) (end 207.38 138.32) (width 0.254) (layer Dolna) (net 17))
+  (segment (start 241.75 116.55) (end 240.2 118.1) (width 0.254) (layer Dolna) (net 17))
+  (segment (start 240.2 118.1) (end 234.225 118.1) (width 0.254) (layer Dolna) (net 17))
+  (segment (start 234.225 118.1) (end 232.5 119.825) (width 0.254) (layer Dolna) (net 17))
+  (segment (start 232.5 119.825) (end 224.3 119.825) (width 0.254) (layer Dolna) (net 17))
+  (segment (start 224.3 119.825) (end 221.625 122.5) (width 0.254) (layer Dolna) (net 17))
+  (segment (start 221.625 122.5) (end 221.625 127.25) (width 0.254) (layer Dolna) (net 17))
+  (segment (start 221.625 127.25) (end 218.725 130.15) (width 0.254) (layer Dolna) (net 17))
+  (segment (start 240.35 118.025) (end 240.35 119.35) (width 0.254) (layer Gorna) (net 17))
+  (via (at 241.825 116.55) (size 0.889) (layers Gorna Dolna) (net 17))
+  (segment (start 240.35 118.025) (end 241.825 116.55) (width 0.254) (layer Gorna) (net 17))
   (segment (start 241.825 116.55) (end 241.75 116.55) (width 0.254) (layer Dolna) (net 17))
-  (segment (start 240.35 118.025) (end 241.825 116.55) (width 0.254) (layer Gorna) (net 17))
-  (via (at 241.825 116.55) (size 0.889) (layers Gorna Dolna) (net 17))
-  (segment (start 240.35 119.35) (end 240.35 118.025) (width 0.254) (layer Gorna) (net 17))
-  (segment (start 207.38 131.695) (end 207.38 145) (width 0.254) (layer Dolna) (net 17))
-  (segment (start 208.925 130.15) (end 207.38 131.695) (width 0.254) (layer Dolna) (net 17))
-  (segment (start 218.725 130.15) (end 208.925 130.15) (width 0.254) (layer Dolna) (net 17))
-  (segment (start 221.625 127.25) (end 218.725 130.15) (width 0.254) (layer Dolna) (net 17))
-  (segment (start 221.625 122.5) (end 221.625 127.25) (width 0.254) (layer Dolna) (net 17))
-  (segment (start 224.3 119.825) (end 221.625 122.5) (width 0.254) (layer Dolna) (net 17))
-  (segment (start 232.5 119.825) (end 224.3 119.825) (width 0.254) (layer Dolna) (net 17))
-  (segment (start 234.225 118.1) (end 232.5 119.825) (width 0.254) (layer Dolna) (net 17))
-  (segment (start 240.2 118.1) (end 234.225 118.1) (width 0.254) (layer Dolna) (net 17))
-  (segment (start 241.75 116.55) (end 240.2 118.1) (width 0.254) (layer Dolna) (net 17))
+  (segment (start 216.45 130.15) (end 218.725 130.15) (width 0.254) (layer Dolna) (net 17))
+  (segment (start 215.55 130.15) (end 216.45 130.15) (width 0.254) (layer Dolna) (net 17))
+  (segment (start 207.38 138.32) (end 215.55 130.15) (width 0.254) (layer Dolna) (net 17))
   (segment (start 233.35 126.85) (end 229.351 126.85) (width 0.254) (layer Gorna) (net 18))
   (segment (start 244.099 110.75) (end 244.099 106.802) (width 0.254) (layer Gorna) (net 19))
@@
   (segment (start 237.85 135.9) (end 237.85 133.35) (width 0.254) (layer Gorna) (net 22))
   (segment (start 238.35 136.4) (end 237.85 135.9) (width 0.254) (layer Gorna) (net 22))
+  (segment (start 213.3875 136.8125) (end 216.2125 136.8125) (width 0.254) (layer Gorna) (net 23))
+  (segment (start 221.25 137.45) (end 221.25 134.35) (width 0.254) (layer Dolna) (net 23))
+  (segment (start 221.2 137.5) (end 221.25 137.45) (width 0.254) (layer Dolna) (net 23))
+  (via (at 221.2 137.5) (size 0.889) (layers Gorna Dolna) (net 23))
+  (segment (start 216.9 137.5) (end 221.2 137.5) (width 0.254) (layer Gorna) (net 23))
+  (segment (start 216.2125 136.8125) (end 216.9 137.5) (width 0.254) (layer Gorna) (net 23))
+  (segment (start 206.025 129.475) (end 209.2 132.65) (width 0.254) (layer Dolna) (net 23))
+  (segment (start 206.025 129.475) (end 206.025 113.45) (width 0.254) (layer Dolna) (net 23))
+  (segment (start 206.025 113.45) (end 209.92 109.555) (width 0.254) (layer Dolna) (net 23))
+  (segment (start 209.92 100) (end 209.92 109.555) (width 0.254) (layer Dolna) (net 23))
+  (segment (start 209.325 132.75) (end 209.2 132.75) (width 0.254) (layer Gorna) (net 23))
+  (via (at 209.2 132.75) (size 0.889) (layers Gorna Dolna) (net 23))
+  (segment (start 209.325 132.75) (end 213.3875 136.8125) (width 0.254) (layer Gorna) (net 23))
+  (segment (start 213.3875 136.8125) (end 213.4 136.825) (width 0.254) (layer Gorna) (net 23))
+  (segment (start 209.2 132.65) (end 209.2 132.75) (width 0.254) (layer Dolna) (net 23))
   (segment (start 221.25 134.35) (end 221.25 133.6) (width 0.254) (layer Dolna) (net 23))
+  (segment (start 221.25 133.6) (end 221.475 133.375) (width 0.254) (layer Dolna) (net 23))
+  (segment (start 223.1 133.3) (end 223.3625 133.5625) (width 0.254) (layer Gorna) (net 23))
+  (via (at 221.475 133.375) (size 0.889) (layers Gorna Dolna) (net 23))
+  (segment (start 221.55 133.3) (end 221.475 133.375) (width 0.254) (layer Gorna) (net 23))
   (segment (start 223.1 133.3) (end 221.55 133.3) (width 0.254) (layer Gorna) (net 23))
-  (segment (start 221.55 133.3) (end 221.475 133.375) (width 0.254) (layer Gorna) (net 23))
-  (via (at 221.475 133.375) (size 0.889) (layers Gorna Dolna) (net 23))
-  (segment (start 223.1 133.3) (end 223.3625 133.5625) (width 0.254) (layer Gorna) (net 23))
-  (segment (start 221.25 133.6) (end 221.475 133.375) (width 0.254) (layer Dolna) (net 23))
-  (segment (start 221.275 136.825) (end 213.375 136.825) (width 0.254) (layer Gorna) (net 23))
-  (segment (start 209.92 109.555) (end 209.92 100) (width 0.254) (layer Dolna) (net 23))
-  (segment (start 206.025 113.45) (end 209.92 109.555) (width 0.254) (layer Dolna) (net 23))
-  (segment (start 206.025 129.475) (end 206.025 113.45) (width 0.254) (layer Dolna) (net 23))
-  (segment (start 206.575 130.025) (end 206.025 129.475) (width 0.254) (layer Dolna) (net 23))
-  (via (at 206.575 130.025) (size 0.889) (layers Gorna Dolna) (net 23))
-  (segment (start 213.375 136.825) (end 206.575 130.025) (width 0.254) (layer Gorna) (net 23))
+  (segment (start 213.4 136.825) (end 213.375 136.825) (width 0.254) (layer Gorna) (net 23))
   (segment (start 249.1 134.45) (end 249.425 134.775) (width 0.254) (layer Gorna) (net 23))
   (segment (start 238.85 133) (end 240.3 134.45) (width 0.254) (layer Gorna) (net 23))
@@
   (segment (start 249.425 138.35) (end 248.175 139.6) (width 0.254) (layer Gorna) (net 23))
   (segment (start 249.425 134.775) (end 249.425 138.35) (width 0.254) (layer Gorna) (net 23))
-  (segment (start 221.275 136.825) (end 221.125 136.825) (width 0.254) (layer Gorna) (net 23))
-  (via (at 221.275 136.825) (size 0.889) (layers Gorna Dolna) (net 23))
-  (segment (start 221.25 136.8) (end 221.275 136.825) (width 0.254) (layer Dolna) (net 23))
   (segment (start 221.25 134.3) (end 221.25 134.35) (width 0.254) (layer Dolna) (net 23))
-  (segment (start 221.25 134.35) (end 221.25 136.8) (width 0.254) (layer Dolna) (net 23))
   (segment (start 223.3625 133.5625) (end 223.35 133.55) (width 0.254) (layer Gorna) (net 23))
   (segment (start 249.1 133.85) (end 249.275 133.85) (width 0.254) (layer Gorna) (net 24))
@@
   (segment (start 231.4 123.625) (end 230.925 123.625) (width 0.254) (layer Gorna) (net 35))
   (segment (start 232.125 124.35) (end 231.4 123.625) (width 0.254) (layer Gorna) (net 35))
-  (zone (net 13) (net_name GND) (layer Gorna) (hatch edge 0.508)
-    (connect_pads yes (clearance 0.254))
+  (zone (net 13) (net_name GND) (layer Dolna) (hatch edge 0.508)
+    (connect_pads (clearance 0.254))
     (min_thickness 0.254)
     (fill (arc_segments 32) (thermal_gap 0.508) (thermal_bridge_width 0.508))
     (polygon
       (pts
-        (xy 272.5 148) (xy 197.75 148) (xy 197.75 97.5) (xy 272.5 97.5)
+        (xy 197.7 97.3) (xy 272.5 97.35) (xy 272.45 148.05) (xy 197.75 148.05) (xy 197.7 97.3)
       )
     )
   )
-  (zone (net 13) (net_name GND) (layer Dolna) (hatch edge 0.508)
-    (connect_pads yes (clearance 0.254))
+  (zone (net 13) (net_name GND) (layer Gorna) (hatch edge 0.508)
+    (connect_pads (clearance 0.254))
     (min_thickness 0.254)
     (fill (arc_segments 32) (thermal_gap 0.508) (thermal_bridge_width 0.508))
     (polygon
       (pts
-        (xy 272.5 148) (xy 197.75 148) (xy 197.75 97.5) (xy 272.5 97.5)
+        (xy 272.5 97.35) (xy 272.45 148.05) (xy 197.75 148.05) (xy 197.7 97.3)
       )
     )
