File: Vehicle_car.sch (KiCad schematic (older format))
At the start: 1 part

Commit message: Schematic continue
Parts:
- added C? (x2): 20pF, ~, symbol C
- added C?: 0.33uF, ~, symbol C
- added C?: 0.1uF, ~, symbol C
- added C? (x2): 10uF, ~, symbol CP1
- added C?: 100nF, ~, symbol C
- added D?: GREEN, ~, symbol LED
- added P?: Supply, ~, symbol CONN_2
- added R?: 0R, ~, symbol R
- added R?: 660R, ~, symbol R
- added U?: LM7805, ~, symbol LM7805
- added U?: LD1117DT33, ~, symbol LD1117DT33
- added X?: 8M, ~, symbol CRYSTAL
Connections:
- net labels added: 3V3, 5V, 9V, GND, OSC_IN, OSC_OUT
- wire segments 0 -> 37

Commit message: GPS, Bluetooth, SWD on schematic
Parts:
- added C? (x2): 100nF, ~, symbol C
- added P?: SWD, ~, symbol CONN_6
- added P?: BLUETOOTH, ~, symbol CONN_7X2
- added P?: GPS, ~, symbol CONN_4
- added R?: 100K, ~, symbol R
- added R?: 510R, ~, symbol R
- added SW?: SW_PUSH_4PIN, ~, symbol SW_PUSH_4PIN
- P?: value Supply -> SUPPLY
Connections:
- net labels added: BLUETOOTH_RX, BLUETOOTH_TX, GPS_RX, GPS_TX, NRST, SWDCLK, SWDIO, SWDO
- wire segments 37 -> 92
Other:
- note added: "Not fitted"
- note added: "OSCILATOR"
- note added: "RESET"
- note added: "SUPPLY\n"
- moved on the sheet: C?, D?, P?, R?, U?, X?

Commit message: Color sensor and TB6612 create
Parts:
- removed C?: 0.33uF, ~, symbol C
- removed C?: 0.1uF, ~, symbol C
- removed P?: BLUETOOTH, ~, symbol CONN_7X2
- removed U?: LM7805, ~, symbol LM7805
- added C? (x2): 100nF, ~, symbol C
- added P?: COLOR_1, ~, symbol CONN_8
- added P?: COLOR_2, ~, symbol CONN_8
- added U?: TB6612, MODULE, symbol TB6612
Connections:
- net labels added: AIN1, AIN2, AO1, AO2, BIN1, BIN2, BO1, BO2, EOa, EOb, OUTa, OUTb, PWMA, PWMB, S0a, S0b, S1a, S1b
- wire segments 92 -> 139
Other:
- moved on the sheet: C?

Commit message: Bluetooth, connect to STM
Parts:
- added D? (x4): GREEN, ~, symbol LED
- added P?: BLUETOOTH, ~, symbol CONN_7X2
- added P?: MOTOR 1, ~, symbol CONN_2
- added P?: MOTOR 2, ~, symbol CONN_2
- added R? (x4): 660R, ~, symbol R
Connections:
- wire segments 139 -> 169
Other:
- note added: "CONNECTORS\n\n\n"
- note added: "H_BRDGE\n"
- note added: "STM32F00\n\n"
- note added: "VCC"
- note added: "VCC_TB\n"
- note added: "VM_TB\n"
- moved on the sheet: P?, R?, U?

Commit message: footprint and finish schematic
Parts:
- removed R?: 0R, ~, symbol R
- added P9: GND, ~, symbol CONN_1
- D1: renamed from D?; value GREEN -> RED
- D4, D5: renamed from D?; value GREEN -> BLUE
- R2, R3: renamed from R?; value 660R -> 330R
- gave numbers to parts that had none: 29
Connections:
- net labels added: LED1, LED2, LED3, LED4
- net labels removed: 5V
- wire segments 169 -> 178
Other:
- note added: "LEDS\n\n"
- moved on the sheet: D2, D3, D4, D5, R2, R3, R4, R5

Commit message: ,,
Connections:
- net labels added: +3,3V, +9V
- net labels removed: 9V
Changed lines of the file:
@@
 Sheet 1 1
 Title ""
-Date "4 nov 2014"
+Date "7 nov 2014"
 Rev ""
 Comp ""
@@
 Comment4 ""
 $EndDescr
-$Comp
-L STM32F100RB U3
-U 1 1 5447853B
-P 8400 4750
-F 0 "U3" H 7100 6700 60  0000 C CNN
-F 1 "STM32F100RB" H 9450 2850 60  0000 C CNN
-F 2 "LQFP64" H 8400 4750 40  0000 C CIN
-F 3 "~" H 8400 4750 60  0000 C CNN
-	1    8400 4750
-	1    0    0    -1
-$EndComp
 $Comp
 L C C9
@@
 	1    0    0    -1
 $EndComp
-Text GLabel 2500 6650 2    39   Input ~ 0
-3V3
 $Comp
 L R R1
@@
 	1    0    0    -1
 $EndComp
-Text GLabel 1250 5850 2    39   Input ~ 0
-9V
 Text GLabel 6800 3600 0    39   Input ~ 0
 OSC_IN
@@
 Text GLabel 5250 6700 2    39   Input ~ 0
 OSC_IN
-Text GLabel 8400 2500 1    39   Input ~ 0
-3V3
 $Comp
 L GND #PWR06
@@
 	1    0    0    -1
 $EndComp
-Text GLabel 1850 5750 1    39   Input ~ 0
-3V3
 Text GLabel 6800 3150 0    39   Input ~ 0
 NRST
@@
 	0    -1   -1   0
 $EndComp
-Text GLabel 5450 5450 2    39   Input ~ 0
-3V3
 Text Notes 4950 5600 0    39   ~ 0
 Not fitted
-Text GLabel 6800 4200 0    39   Input ~ 0
-3V3
 $Comp
 L R R8
@@
 	1    0    0    -1
 $EndComp
-Text GLabel 1150 3350 1    39   Input ~ 0
-3V3
 Text GLabel 1150 3550 2    39   Input ~ 0
 SWDCLK
@@
 Connection ~ 2100 6850
 Wire Wire Line
-	2300 6850 2300 6650
-Wire Wire Line
-	2300 6650 2500 6650
-Connection ~ 2300 6850
-Wire Wire Line
 	2900 6850 3000 6850
 Wire Wire Line
@@
 	3500 6850 3500 6950
 Wire Wire Line
-	1250 5850 1100 5850
+	1100 5850 1300 5850
 Wire Wire Line
 	1300 6050 1300 6150
@@
 Wire Wire Line
 	5450 5450 5300 5450
-Wire Wire Line
-	6900 4200 6800 4200
 Wire Wire Line
 	6900 3350 6800 3350
@@
 Wire Wire Line
 	1200 4750 1200 4650
-Text GLabel 1200 4650 1    39   Input ~ 0
-3V3
 Wire Wire Line
 	1100 4850 1200 4850
@@
 	1    0    0    -1
 $EndComp
-Text GLabel 1850 750  1    39   Input ~ 0
-3V3
 Wire Wire Line
 	1900 850  1900 950
@@
 	2100 750  2100 950
 Connection ~ 2100 850
-Text GLabel 2100 750  1    39   Input ~ 0
-9V
 Wire Wire Line
 	1000 1450 900  1450
@@
 Wire Wire Line
 	2250 6250 2250 6400
-Text GLabel 2250 5750 1    39   Input ~ 0
-9V
 Wire Wire Line
 	2250 5850 2250 5750
@@
 	1    0    0    -1
 $EndComp
-Text GLabel 2650 5750 1    39   Input ~ 0
-3V3
 Wire Wire Line
 	2650 5850 2650 5750
@@
 	-1   0    0    -1
 $EndComp
-Text GLabel 2450 3150 1    39   Input ~ 0
-3V3
 Wire Wire Line
 	2350 3250 2450 3250
@@
 Text GLabel 2450 3550 2    39   Input ~ 0
 S1a
-Text GLabel 2700 3550 1    39   Input ~ 0
-3V3
 Wire Wire Line
 	2350 3650 2700 3650
@@
 Text GLabel 2450 3950 2    39   Input ~ 0
 OUTa
-Text GLabel 2450 4300 1    39   Input ~ 0
-3V3
 Wire Wire Line
 	2350 4400 2450 4400
@@
 Text GLabel 2450 4700 2    39   Input ~ 0
 S1b
-Text GLabel 2750 4700 1    39   Input ~ 0
-3V3
 Wire Wire Line
 	2350 4800 2750 4800
@@
 Wire Wire Line
 	3450 4400 3450 4500
-Text GLabel 3450 4400 1    39   Input ~ 0
-3V3
 $Comp
 L GND #PWR019
@@
 Wire Wire Line
 	4500 4500 4350 4500
-Text GLabel 3450 4600 0    39   Input ~ 0
+Text GLabel 3450 4700 0    39   Input ~ 0
 BLUETOOTH_TX
-Wire Wire Line
-	3550 4600 3450 4600
 Wire Wire Line
 	4350 4600 4450 4600
@@
 Wire Wire Line
 	750  6850 750  6750
-Text GLabel 750  6750 1    39   Input ~ 0
-9V
+Wire Wire Line
+	6900 4200 6800 4200
+Text GLabel 6800 4200 0    39   Input ~ 0
+3V3
+$Comp
+L STM32F100RB U3
+U 1 1 5447853B
+P 8400 4750
+F 0 "U3" H 7100 6700 60  0000 C CNN
+F 1 "STM32F100RB" H 9450 2850 60  0000 C CNN
+F 2 "LQFP64" H 8400 4750 40  0000 C CIN
+F 3 "~" H 8400 4750 60  0000 C CNN
+	1    8400 4750
+	1    0    0    -1
+$EndComp
+$Comp
+L +9V #PWR022
+U 1 1 545B7806
+P 1300 5750
+F 0 "#PWR022" H 1300 5720 20  0001 C CNN
+F 1 "+9V" H 1300 5860 30  0000 C CNN
+F 2 "~" H 1300 5750 60  0000 C CNN
+F 3 "~" H 1300 5750 60  0000 C CNN
+	1    1300 5750
+	1    0    0    -1
+$EndComp
+$Comp
+L +9V #PWR023
+U 1 1 545B7813
+P 750 6750
+F 0 "#PWR023" H 750 6720 20  0001 C CNN
+F 1 "+9V" H 750 6860 30  0000 C CNN
+F 2 "~" H 750 6750 60  0000 C CNN
+F 3 "~" H 750 6750 60  0000 C CNN
+	1    750  6750
+	1    0    0    -1
+$EndComp
+Wire Wire Line
+	1300 5850 1300 5750
+$Comp
+L +3,3V #PWR?
+U 1 1 545B7A8E
+P 2300 6700
+F 0 "#PWR?" H 2300 6660 30  0001 C CNN
+F 1 "+3,3V" H 2300 6810 30  0000 C CNN
+F 2 "~" H 2300 6700 60  0000 C CNN
+F 3 "~" H 2300 6700 60  0000 C CNN
+	1    2300 6700
+	1    0    0    -1
+$EndComp
+Wire Wire Line
+	2300 6850 2300 6700
+Connection ~ 2300 6850
+$Comp
+L +3,3V #PWR?
+U 1 1 545B7B84
+P 1850 5750
+F 0 "#PWR?" H 1850 5710 30  0001 C CNN
+F 1 "+3,3V" H 1850 5860 30  0000 C CNN
+F 2 "~" H 1850 5750 60  0000 C CNN
+F 3 "~" H 1850 5750 60  0000 C CNN
+	1    1850 5750
+	1    0    0    -1
+$EndComp
+$Comp
+L +3,3V #PWR?
+U 1 1 545B7B8A
+P 2650 5750
+F 0 "#PWR?" H 2650 5710 30  0001 C CNN
+F 1 "+3,3V" H 2650 5860 30  0000 C CNN
+F 2 "~" H 2650 5750 60  0000 C CNN
+F 3 "~" H 2650 5750 60  0000 C CNN
+	1    2650 5750
+	1    0    0    -1
+$EndComp
+$Comp
+L +9V #PWR?
+U 1 1 545B7B90
+P 2250 5750
+F 0 "#PWR?" H 2250 5720 20  0001 C CNN
+F 1 "+9V" H 2250 5860 30  0000 C CNN
+F 2 "~" H 2250 5750 60  0000 C CNN
+F 3 "~" H 2250 5750 60  0000 C CNN
+	1    2250 5750
+	1    0    0    -1
+$EndComp
+$Comp
+L +3,3V #PWR?
+U 1 1 545B7BB4
+P 5450 5450
+F 0 "#PWR?" H 5450 5410 30  0001 C CNN
+F 1 "+3,3V" H 5450 5560 30  0000 C CNN
+F 2 "~" H 5450 5450 60  0000 C CNN
+F 3 "~" H 5450 5450 60  0000 C CNN
+	1    5450 5450
+	0    1    1    0
+$EndComp
+$Comp
+L +3,3V #PWR?
+U 1 1 545B7D17
+P 1200 4650
+F 0 "#PWR?" H 1200 4610 30  0001 C CNN
+F 1 "+3,3V" H 1200 4760 30  0000 C CNN
+F 2 "~" H 1200 4650 60  0000 C CNN
+F 3 "~" H 1200 4650 60  0000 C CNN
+	1    1200 4650
+	1    0    0    -1
+$EndComp
+$Comp
+L +3,3V #PWR?
+U 1 1 545B7D1D
+P 2450 4300
+F 0 "#PWR?" H 2450 4260 30  0001 C CNN
+F 1 "+3,3V" H 2450 4410 30  0000 C CNN
+F 2 "~" H 2450 4300 60  0000 C CNN
+F 3 "~" H 2450 4300 60  0000 C CNN
+	1    2450 4300
+	1    0    0    -1
+$EndComp
+$Comp
+L +3,3V #PWR?
+U 1 1 545B7D23
+P 2750 4700
+F 0 "#PWR?" H 2750 4660 30  0001 C CNN
+F 1 "+3,3V" H 2750 4810 30  0000 C CNN
+F 2 "~" H 2750 4700 60  0000 C CNN
+F 3 "~" H 2750 4700 60  0000 C CNN
+	1    2750 4700
+	1    0    0    -1
+$EndComp
+$Comp
+L +3,3V #PWR?
+U 1 1 545B7D29
+P 3450 4400
+F 0 "#PWR?" H 3450 4360 30  0001 C CNN
+F 1 "+3,3V" H 3450 4510 30  0000 C CNN
+F 2 "~" H 3450 4400 60  0000 C CNN
+F 3 "~" H 3450 4400 60  0000 C CNN
+	1    3450 4400
+	1    0    0    -1
+$EndComp
+$Comp
+L +3,3V #PWR?
+U 1 1 545B7D57
+P 2450 3150
+F 0 "#PWR?" H 2450 3110 30  0001 C CNN
+F 1 "+3,3V" H 2450 3260 30  0000 C CNN
+F 2 "~" H 2450 3150 60  0000 C CNN
+F 3 "~" H 2450 3150 60  0000 C CNN
+	1    2450 3150
+	1    0    0    -1
+$EndComp
+$Comp
+L +3,3V #PWR?
+U 1 1 545B7D5D
+P 2700 3550
+F 0 "#PWR?" H 2700 3510 30  0001 C CNN
+F 1 "+3,3V" H 2700 3660 30  0000 C CNN
+F 2 "~" H 2700 3550 60  0000 C CNN
+F 3 "~" H 2700 3550 60  0000 C CNN
+	1    2700 3550
+	1    0    0    -1
+$EndComp
+$Comp
+L +3,3V #PWR?
+U 1 1 545B7D63
+P 1150 3350
+F 0 "#PWR?" H 1150 3310 30  0001 C CNN
+F 1 "+3,3V" H 1150 3460 30  0000 C CNN
+F 2 "~" H 1150 3350 60  0000 C CNN
+F 3 "~" H 1150 3350 60  0000 C CNN
+	1    1150 3350
+	1    0    0    -1
+$EndComp
+$Comp
+L +3,3V #PWR?
+U 1 1 545B7D87
+P 1850 750
+F 0 "#PWR?" H 1850 710 30  0001 C CNN
+F 1 "+3,3V" H 1850 860 30  0000 C CNN
+F 2 "~" H 1850 750 60  0000 C CNN
+F 3 "~" H 1850 750 60  0000 C CNN
+	1    1850 750
+	1    0    0    -1
+$EndComp
+$Comp
+L +9V #PWR?
+U 1 1 545B7D8D
+P 2100 750
+F 0 "#PWR?" H 2100 720 20  0001 C CNN
+F 1 "+9V" H 2100 860 30  0000 C CNN
+F 2 "~" H 2100 750 60  0000 C CNN
+F 3 "~" H 2100 750 60  0000 C CNN
+	1    2100 750
+	1    0    0    -1
+$EndComp
+$Comp
+L +3,3V #PWR?
+U 1 1 545B7DA7
+P 8400 2500
+F 0 "#PWR?" H 8400 2460 30  0001 C CNN
+F 1 "+3,3V" H 8400 2610 30  0000 C CNN
+F 2 "~" H 8400 2500 60  0000 C CNN
+F 3 "~" H 8400 2500 60  0000 C CNN
+	1    8400 2500
+	1    0    0    -1
+$EndComp
+Wire Wire Line
+	3550 4700 3450 4700
 $EndSCHEMATC

Commit message: Finished schematic. Not checked yet
Parts:
- added P10: Length_sen, ~, symbol CONN_4
Connections:
- net labels added: SEN_EN, SEN_OUT
- wire segments 178 -> 186
Other:
- moved on the sheet: P9
Changed lines of the file:
@@
 Sheet 1 1
 Title ""
-Date "7 nov 2014"
+Date "8 nov 2014"
 Rev ""
 Comp ""
@@
 L CONN_1 P9
 U 1 1 5454D0D9
-P 4550 3900
-F 0 "P9" H 4630 3900 40  0000 L CNN
-F 1 "GND" H 4550 3955 30  0001 C CNN
-F 2 "~" H 4550 3900 60  0000 C CNN
-F 3 "~" H 4550 3900 60  0000 C CNN
-	1    4550 3900
+P 4500 3900
+F 0 "P9" H 4580 3900 40  0000 L CNN
+F 1 "GND" H 4500 3955 30  0001 C CNN
+F 2 "~" H 4500 3900 60  0000 C CNN
+F 3 "~" H 4500 3900 60  0000 C CNN
+	1    4500 3900
 	-1   0    0    1
 $EndComp
 Wire Wire Line
-	4700 3900 4800 3900
-Wire Wire Line
-	4800 3900 4800 4000
+	4650 3900 4750 3900
+Wire Wire Line
+	4750 3900 4750 4000
 $Comp
 L GND #PWR021
 U 1 1 5454D1D1
-P 4800 4000
-F 0 "#PWR021" H 4800 4000 30  0001 C CNN
-F 1 "GND" H 4800 3930 30  0001 C CNN
-F 2 "~" H 4800 4000 60  0000 C CNN
-F 3 "~" H 4800 4000 60  0000 C CNN
-	1    4800 4000
+P 4750 4000
+F 0 "#PWR021" H 4750 4000 30  0001 C CNN
+F 1 "GND" H 4750 3930 30  0001 C CNN
+F 2 "~" H 4750 4000 60  0000 C CNN
+F 3 "~" H 4750 4000 60  0000 C CNN
+	1    4750 4000
 	1    0    0    -1
 $EndComp
@@
 	1300 5850 1300 5750
 $Comp
-L +3,3V #PWR?
+L +3,3V #PWR024
 U 1 1 545B7A8E
 P 2300 6700
-F 0 "#PWR?" H 2300 6660 30  0001 C CNN
+F 0 "#PWR024" H 2300 6660 30  0001 C CNN
 F 1 "+3,3V" H 2300 6810 30  0000 C CNN
 F 2 "~" H 2300 6700 60  0000 C CNN
@@
 Connection ~ 2300 6850
 $Comp
-L +3,3V #PWR?
+L +3,3V #PWR025
 U 1 1 545B7B84
 P 1850 5750
-F 0 "#PWR?" H 1850 5710 30  0001 C CNN
+F 0 "#PWR025" H 1850 5710 30  0001 C CNN
 F 1 "+3,3V" H 1850 5860 30  0000 C CNN
 F 2 "~" H 1850 5750 60  0000 C CNN
@@
 $EndComp
 $Comp
-L +3,3V #PWR?
+L +3,3V #PWR026
 U 1 1 545B7B8A
 P 2650 5750
-F 0 "#PWR?" H 2650 5710 30  0001 C CNN
+F 0 "#PWR026" H 2650 5710 30  0001 C CNN
 F 1 "+3,3V" H 2650 5860 30  0000 C CNN
 F 2 "~" H 2650 5750 60  0000 C CNN
@@
 $EndComp
 $Comp
-L +9V #PWR?
+L +9V #PWR027
 U 1 1 545B7B90
 P 2250 5750
-F 0 "#PWR?" H 2250 5720 20  0001 C CNN
+F 0 "#PWR027" H 2250 5720 20  0001 C CNN
 F 1 "+9V" H 2250 5860 30  0000 C CNN
 F 2 "~" H 2250 5750 60  0000 C CNN
@@
 $EndComp
 $Comp
-L +3,3V #PWR?
+L +3,3V #PWR028
 U 1 1 545B7BB4
 P 5450 5450
-F 0 "#PWR?" H 5450 5410 30  0001 C CNN
+F 0 "#PWR028" H 5450 5410 30  0001 C CNN
 F 1 "+3,3V" H 5450 5560 30  0000 C CNN
 F 2 "~" H 5450 5450 60  0000 C CNN
@@
 $EndComp
 $Comp
-L +3,3V #PWR?
+L +3,3V #PWR029
 U 1 1 545B7D17
 P 1200 4650
-F 0 "#PWR?" H 1200 4610 30  0001 C CNN
+F 0 "#PWR029" H 1200 4610 30  0001 C CNN
 F 1 "+3,3V" H 1200 4760 30  0000 C CNN
 F 2 "~" H 1200 4650 60  0000 C CNN
@@
 $EndComp
 $Comp
-L +3,3V #PWR?
+L +3,3V #PWR030
 U 1 1 545B7D1D
 P 2450 4300
-F 0 "#PWR?" H 2450 4260 30  0001 C CNN
+F 0 "#PWR030" H 2450 4260 30  0001 C CNN
 F 1 "+3,3V" H 2450 4410 30  0000 C CNN
 F 2 "~" H 2450 4300 60  0000 C CNN
@@
 $EndComp
 $Comp
-L +3,3V #PWR?
+L +3,3V #PWR031
 U 1 1 545B7D23
 P 2750 4700
-F 0 "#PWR?" H 2750 4660 30  0001 C CNN
+F 0 "#PWR031" H 2750 4660 30  0001 C CNN
 F 1 "+3,3V" H 2750 4810 30  0000 C CNN
 F 2 "~" H 2750 4700 60  0000 C CNN
@@
 $EndComp
 $Comp
-L +3,3V #PWR?
+L +3,3V #PWR032
 U 1 1 545B7D29
 P 3450 4400
-F 0 "#PWR?" H 3450 4360 30  0001 C CNN
+F 0 "#PWR032" H 3450 4360 30  0001 C CNN
 F 1 "+3,3V" H 3450 4510 30  0000 C CNN
 F 2 "~" H 3450 4400 60  0000 C CNN
@@
 $EndComp
 $Comp
-L +3,3V #PWR?
+L +3,3V #PWR033
 U 1 1 545B7D57
 P 2450 3150
-F 0 "#PWR?" H 2450 3110 30  0001 C CNN
+F 0 "#PWR033" H 2450 3110 30  0001 C CNN
 F 1 "+3,3V" H 2450 3260 30  0000 C CNN
 F 2 "~" H 2450 3150 60  0000 C CNN
@@
 $EndComp
 $Comp
-L +3,3V #PWR?
+L +3,3V #PWR034
 U 1 1 545B7D5D
 P 2700 3550
-F 0 "#PWR?" H 2700 3510 30  0001 C CNN
+F 0 "#PWR034" H 2700 3510 30  0001 C CNN
 F 1 "+3,3V" H 2700 3660 30  0000 C CNN
 F 2 "~" H 2700 3550 60  0000 C CNN
@@
 $EndComp
 $Comp
-L +3,3V #PWR?
+L +3,3V #PWR035
 U 1 1 545B7D63
 P 1150 3350
-F 0 "#PWR?" H 1150 3310 30  0001 C CNN
+F 0 "#PWR035" H 1150 3310 30  0001 C CNN
 F 1 "+3,3V" H 1150 3460 30  0000 C CNN
 F 2 "~" H 1150 3350 60  0000 C CNN
@@
 $EndComp
 $Comp
-L +3,3V #PWR?
+L +3,3V #PWR036
 U 1 1 545B7D87
 P 1850 750
-F 0 "#PWR?" H 1850 710 30  0001 C CNN
+F 0 "#PWR036" H 1850 710 30  0001 C CNN
 F 1 "+3,3V" H 1850 860 30  0000 C CNN
 F 2 "~" H 1850 750 60  0000 C CNN
@@
 $EndComp
 $Comp
-L +9V #PWR?
+L +9V #PWR037
 U 1 1 545B7D8D
 P 2100 750
-F 0 "#PWR?" H 2100 720 20  0001 C CNN
+F 0 "#PWR037" H 2100 720 20  0001 C CNN
 F 1 "+9V" H 2100 860 30  0000 C CNN
 F 2 "~" H 2100 750 60  0000 C CNN
@@
 $EndComp
 $Comp
-L +3,3V #PWR?
+L +3,3V #PWR038
 U 1 1 545B7DA7
 P 8400 2500
-F 0 "#PWR?" H 8400 2460 30  0001 C CNN
+F 0 "#PWR038" H 8400 2460 30  0001 C CNN
 F 1 "+3,3V" H 8400 2610 30  0000 C CNN
 F 2 "~" H 8400 2500 60  0000 C CNN
@@
 Wire Wire Line
 	3550 4700 3450 4700
+$Comp
+L CONN_4 P10
+U 1 1 545DD0AC
+P 4400 3400
+F 0 "P10" V 4350 3400 50  0000 C CNN
+F 1 "Length_sen" V 4450 3400 50  0000 C CNN
+F 2 "~" H 4400 3400 60  0000 C CNN
+F 3 "~" H 4400 3400 60  0000 C CNN
+	1    4400 3400
+	-1   0    0    -1
+$EndComp
+Wire Wire Line
+	4750 3250 4850 3250
+Wire Wire Line
+	4750 3350 4850 3350
+Wire Wire Line
+	4750 3450 5300 3450
+Wire Wire Line
+	4750 3550 4950 3550
+$Comp
+L GND #PWR039
+U 1 1 545DD486
+P 4950 3650
+F 0 "#PWR039" H 4950 3650 30  0001 C CNN
+F 1 "GND" H 4950 3580 30  0001 C CNN
+F 2 "~" H 4950 3650 60  0000 C CNN
+F 3 "~" H 4950 3650 60  0000 C CNN
+	1    4950 3650
+	1    0    0    -1
+$EndComp
+Wire Wire Line
+	4950 3550 4950 3650
+$Comp
+L +3,3V #PWR040
+U 1 1 545DD661
+P 5300 3350
+F 0 "#PWR040" H 5300 3310 30  0001 C CNN
+F 1 "+3,3V" H 5300 3460 30  0000 C CNN
+F 2 "~" H 5300 3350 60  0000 C CNN
+F 3 "~" H 5300 3350 60  0000 C CNN
+	1    5300 3350
+	1    0    0    -1
+$EndComp
+Text GLabel 4850 3350 2    39   Input ~ 0
+SEN_OUT
+Text GLabel 4850 3250 2    39   Input ~ 0
+SEN_EN
+Wire Wire Line
+	5300 3450 5300 3350
+Wire Wire Line
+	9900 5350 10000 5350
+Text GLabel 10000 5350 2    39   Input ~ 0
+SEN_OUT
+Wire Wire Line
+	9900 5450 10000 5450
+Text GLabel 10000 5450 2    39   Input ~ 0
+SEN_EN
 $EndSCHEMATC

Commit message: PCB dimension
Parts:
- added DR1: DRILL_6MM_3MM, ~, symbol DRILL_6MM_3MM
- added P11: GND, ~, symbol CONN_1
Connections:
- wire segments 186 -> 188
Changed lines of the file:
@@
 LIBS:stm32
 LIBS:H_Bridge
+LIBS:DRILLS
 LIBS:Vehicle_car-cache
 EELAYER 27 0
@@
 Text GLabel 10000 5450 2    39   Input ~ 0
 SEN_EN
+$Comp
+L DRILL_6MM_3MM DR1
+U 1 1 545E0CFE
+P 6200 1400
+F 0 "DR1" H 6150 1550 60  0000 C CNN
+F 1 "DRILL_6MM_3MM" H 6200 1200 60  0000 C CNN
+F 2 "~" H 6200 1400 60  0000 C CNN
+F 3 "~" H 6200 1400 60  0000 C CNN
+	1    6200 1400
+	1    0    0    -1
+$EndComp
+$Comp
+L CONN_1 P11
+U 1 1 545EAACE
+P 4500 4150
+F 0 "P11" H 4580 4150 40  0000 L CNN
+F 1 "GND" H 4500 4205 30  0001 C CNN
+F 2 "~" H 4500 4150 60  0000 C CNN
+F 3 "~" H 4500 4150 60  0000 C CNN
+	1    4500 4150
+	-1   0    0    1
+$EndComp
+Wire Wire Line
+	4650 4150 4750 4150
+Wire Wire Line
+	4750 4150 4750 4250
+$Comp
+L GND #PWR041
+U 1 1 545EAAD6
+P 4750 4250
+F 0 "#PWR041" H 4750 4250 30  0001 C CNN
+F 1 "GND" H 4750 4180 30  0001 C CNN
+F 2 "~" H 4750 4250 60  0000 C CNN
+F 3 "~" H 4750 4250 60  0000 C CNN
+	1    4750 4250
+	1    0    0    -1
+$EndComp
 $EndSCHEMATC
