File: Vehicle_car.sch (KiCad schematic (older format))
At the start: 38 parts, among them P1 SWD, P10 Length_sen, P11 GND, P2 GPS, P3 SUPPLY, P4 COLOR_1, P5 COLOR_2, P6 MOTOR 1, P7 MOTOR 2, P8 BLUETOOTH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

Commit message: finished PCB arrangement elements
Parts:
- added C10, C11, C12, C13, C14: 100nF, ~, symbol C
Connections:
- net labels added: LEDa, LEDb
- net labels removed: EOa, EOb
- wire segments 188 -> 196
Other:
- note added: "VCC_uP\n"
- note removed: "VCC"
- moved on the sheet: C5, C6

Commit message: Started connect pads
Parts:
- removed D2, D3: GREEN, ~, symbol LED
- removed D4, D5: BLUE, ~, symbol LED
- removed R2, R3: 330R, ~, symbol R
- removed R4, R5: 660R, ~, symbol R
Connections:
- wire segments 196 -> 185
Other:
- note added: "DRILL\n\n"
- note removed: "LEDS\n\n"

Commit message: Finish PCB
Connections:
- net labels removed: 3V3, LED1, LED2, LED3, LED4
- wire segments 185 -> 182
Changed lines of the file:
@@
 Sheet 1 1
 Title ""
-Date "24 nov 2014"
+Date "26 nov 2014"
 Rev ""
 Comp ""
@@
 Text Notes 2550 700  0    59   ~ 12
 H_BRDGE\n
-Wire Wire Line
-	9900 6050 10000 6050
-Wire Wire Line
-	9900 6150 10000 6150
-Wire Wire Line
-	9900 6250 10000 6250
-Wire Wire Line
-	9900 6350 10000 6350
-Text GLabel 10000 6050 2    39   Input ~ 0
-LED1
-Text GLabel 10000 6150 2    39   Input ~ 0
-LED2
-Text GLabel 10000 6250 2    39   Input ~ 0
-LED3
-Text GLabel 10000 6350 2    39   Input ~ 0
-LED4
 Wire Notes Line
 	5750 550  5750 2200
@@
 	750  6850 750  6750
 Wire Wire Line
-	6900 4200 6800 4200
-Text GLabel 6800 4200 0    39   Input ~ 0
-3V3
+	6500 4200 6900 4200
 $Comp
 L STM32F100RB U3
@@
 Wire Wire Line
 	1600 4950 1600 4800
+$Comp
+L +3,3V #PWR051
+U 1 1 5474EAF4
+P 6500 4150
+F 0 "#PWR051" H 6500 4110 30  0001 C CNN
+F 1 "+3,3V" H 6500 4260 30  0000 C CNN
+F 2 "~" H 6500 4150 60  0000 C CNN
+F 3 "~" H 6500 4150 60  0000 C CNN
+	1    6500 4150
+	1    0    0    -1
+$EndComp
+Wire Wire Line
+	6500 4200 6500 4150
 $EndSCHEMATC
